File: hardware/temperature-v2.kicad_pcb (KiCad board)
At the start: 2 copper layers, 15 x 25 mm, 24 parts, among them P1 CON-SENSOR2, P2 DEBUG, P3 BOOT, U1 XMC11XX24, U2 STS3x-DIS, U3 DRILL, U4 DRILL, U5 DRILL, U6 DRILL

Commit message: specify processor, fix references
Parts:
- U1: value XMC11XX24 -> XMC1100
Changed lines of the file:
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@@
       (effects (font (size 0.3 0.3) (thickness 0.075)))
     )
-    (fp_text value XMC11XX24 (at 0 0.8 225) (layer F.Fab)
+    (fp_text value XMC1100 (at 0 0.8 225) (layer F.Fab)
       (effects (font (size 0.3 0.3) (thickness 0.075)))
     )
